Commit message: add movable model with urdf

File: src/pev_simulation/urdf/test_pev.urdf (robot description, URDF)
Before this commit: robot test_pev, 7 links, 6 joints
Links:
- added link bike_frame; visual box size=1.11 2.21 2.21
- added link rear_wheel; visual cylinder length=0.1 radius=0.36
- link base_footprint: geometry visual cylinder length=0.01 radius=0.36
- link base_link: geometry visual sphere radius=0.1
- link handle: geometry visual cylinder length=0.8 radius=0.02
- link left_wheel: geometry visual cylinder length=0.1 radius=0.36
- link right_wheel: geometry visual cylinder length=0.1 radius=0.36
- link steer_base: geometry visual cylinder length=0.1 radius=0.08
- link steer_link: geometry visual cylinder length=0.1 radius=0.08
Joints:
- added joint baselink_to_frame: type fixed, parent base_link, child bike_frame, origin xyz=0 0.6 0 rpy=0 0 0
- added joint baselink_to_rearwheel: type continuous, parent base_link, child rear_wheel, origin xyz=0 0 0 rpy=0 0 0, axis 1 0 0
- joint baselink_to_basefootprint: origin xyz=0 0 0.36 rpy=0 0 0 -> xyz=0 0 -0.36 rpy=0 0 0
- joint baselink_to_steerbase: axis (none) -> 0 0 1; limit (none) -> lower=-0.548 upper=0.548 effort=1000.0 velocity=0.5; type fixed -> revolute
- joint steerbase_to_hadle: origin xyz=0 1.2 0 rpy=0 0 0 -> xyz=0 0 1.2 rpy=0 0 0
- joint steerbase_to_steerlink: axis (none) -> 0 0 1; limit (none) -> lower=-0.548 upper=0.548 effort=1000.0 velocity=0.5; type fixed -> revolute
- joint steerlink_to_leftwheel: axis (none) -> 1 0 0; type fixed -> continuous
- joint steerlink_to_rightwheel: axis (none) -> 1 0 0; type fixed -> continuous
